Commit message: Sync latest competition release and consolidate documentation
Unify reset control, retain current v2 scene, and consolidate usage, deployment, model adapter and algorithm notes into README.
Include navigation/camera/grasp fixes and project-local runtime helpers; remove obsolete duplicate launchers and reports.
Validation: 89 logic checks passed; full live rounds completed 5/5 in 280.9s and 246.2s.
Local Qwen resources, credentials, generated runtimes and large environment image are excluded.

File: ros_ws/src/yzbot/mybot_description/urdf/camera_gazebo.xacro (robot description, xacro)
@@ -30,10 +30,11 @@
         <gazebo reference="${prefix}_link">
             <sensor type="camera" name="camera_node">
-                <update_rate>10.0</update_rate>
+                <always_on>true</always_on>
+                <update_rate>30.0</update_rate>
                 <camera name="head">
-                    <horizontal_fov>1.5708</horizontal_fov> <!-- 90 degrees -->
+                    <horizontal_fov>1.919862</horizontal_fov> <!-- 110 degrees: retain forward range and see near grasp targets -->
                     <image>
-                        <width>640</width>
-                        <height>360</height>
+                        <width>960</width>
+                        <height>540</height>
                         <format>R8G8B8</format>
                     </image>
@@ -48,4 +49,8 @@
                     </noise>
                 </camera>
+                <plugin name="front_compressed_camera" filename="libcompetition_camera_stream.so">
+                    <topic_name>/${prefix}/image_raw/compressed</topic_name>
+                    <frame_name>${prefix}_link</frame_name>
+                </plugin>
                 <plugin name="gazebo_camera" filename="libgazebo_ros_camera.so">
 				    <ros>

File: ros_ws/src/yzbot/mybot_description/urdf/originbot_with_rgbd_gazebo_arm.xacro (robot description, xacro)
@@ -39,5 +39,6 @@
     </joint>
     <!-- Camera -->
-    <xacro:property name="camera_offset_x" value="${base_length/2+0.02}" />
+    <!-- Keep the lens behind the bumper so a cube 22 cm ahead stays in view. -->
+    <xacro:property name="camera_offset_x" value="0.0" />
     <xacro:property name="camera_offset_y" value="0.16" />
     <xacro:property name="camera_offset_z" value="0.30" />
@@ -76,5 +77,6 @@
     <gazebo reference="camera_mount_link"><material>Gazebo/Black</material></gazebo>
     <joint name="camera_joint" type="fixed">
-        <origin xyz="${camera_offset_x} ${camera_offset_y} ${camera_offset_z}" rpy="0 0.60 -0.35" />
+        <!-- Keep both the near grasp point and the next few metres of floor in view. -->
+        <origin xyz="${camera_offset_x} ${camera_offset_y} ${camera_offset_z}" rpy="0 0.57 -0.35" />
         <parent link="base_link" />
         <child link="camera_link" />
